File: Flight_Computer/RCS_Hardware.kicad_sch (KiCad schematic)
At the start: 55 parts, among them J1 SWD, J2 TYPE-C-31-M-12, J3 SPI, J4 5V, J5 GND, J6 Solenoids, J7 SPI, J8 Conn_01x05_Male, U1 STM32F401CCU6, U2 AMS1117-3.3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

Commit message: Added JLCPCB Part numbers to missing schemas Changed JLCPCB# to LSCS Part Adjusted silkscreen for some labels Added Payload LOGO to back silkscreen Generated manufacturing and assembly files
Parts:
- C1, C15, C16, C20, C23, C5, C6, C7, C8: JLCPCB# C307331 -> (none); LCSC Part (none) -> C307331
- C10, C11: JLCPCB# C52923 -> (none); LCSC Part (none) -> C52923
- C12: JLCPCB# C12530 -> (none); LCSC Part (none) -> C12530
- C13, C14: JLCPCB# C5674 -> (none); LCSC Part (none) -> C5674
- C17, C18: JLCPCB# C466226 -> (none); LCSC Part (none) -> C466226
- C2, C3: JLCPCB# C32949 -> (none); LCSC Part (none) -> C32949
- C21, C24: LCSC Part (none) -> C2655418
- C22: LCSC Part (none) -> C295925
- C4: JLCPCB# C19702 -> (none); LCSC Part (none) -> C19702
- C9: JLCPCB# C15195 -> (none); LCSC Part (none) -> C15195
- D1, D2, D3: JLCPCB# C273598 -> (none); LCSC Part (none) -> C273598
- FB1: JLCPCB# C85831 -> (none); LCSC Part (none) -> C85831
- J2: JLCPCB# C165948 -> (none); LCSC Part (none) -> C165948
- R1, R2: JLCPCB# C25906 -> (none); LCSC Part (none) -> C25906
- R3, R8, R9: JLCPCB# C11702 -> (none); LCSC Part (none) -> C11702
- R4, R7: JLCPCB# C60490 -> (none); LCSC Part (none) -> C60490
- U1: JLCPCB# C79861 -> (none); LCSC Part (none) -> C79861
- U2: JLCPCB# C6186 -> (none); LCSC Part (none) -> C6186
- U4: JLCPCB# C93216 -> (none); LCSC Part (none) -> C93216
- U5: JLCPCB# C82344 -> (none); LCSC Part (none) -> C82344
- U6: LCSC Part (none) -> C24112
- Y1: JLCPCB# C13738 -> (none); LCSC Part (none) -> C13738
- Y2: JLCPCB# C907540 -> (none); LCSC Part (none) -> C907540
